Commit message: ETHZ: fixed flipper position
git-svn-id: https://subversion.dfki.de/nifti/code/ros/stacks/nifti_drivers/trunk/nifti_robot_driver@6351 3189491a-1924-0410-a745-03ab4139b441

File: robot_model/nifti_robot.urdf (robot description, URDF)
Before this commit: robot NIFTi, 16 links, 15 joints
Joints:
- joint front_left_flipper_j: origin xyz=0.25 0.0585 0.0195 rpy=0 0.1937 0 -> xyz=0.25 0.0735 0.0195 rpy=0 0.1937 0
- joint front_right_flipper_j: origin xyz=0.25 -0.0585 0.0195 rpy=0 0.1937 0 -> xyz=0.25 -0.0735 0.0195 rpy=0 0.1937 0
- joint rear_left_flipper_j: origin xyz=-0.25 0.0585 0.0195 rpy=0 2.9479 0 -> xyz=-0.25 0.0735 0.0195 rpy=0 2.9479 0
- joint rear_right_flipper_j: origin xyz=-0.25 -0.0585 0.0195 rpy=0 2.9479 0 -> xyz=-0.25 -0.0735 0.0195 rpy=0 2.9479 0

Commit message: IMU orientation and CAN error message
git-svn-id: https://subversion.dfki.de/nifti/code/ros/stacks/nifti_drivers/trunk/nifti_robot_driver@6747 3189491a-1924-0410-a745-03ab4139b441

File: robot_model/nifti_robot.urdf (robot description, URDF)
Before this commit: robot NIFTi, 16 links, 15 joints
Joints:
- joint imu_j: origin xyz=0 0 0.1694 rpy=0 0 0 -> xyz=0 0 0.1694 rpy=0 0 -1.5707963267

Commit message: ETHZ: updated robot model
git-svn-id: https://subversion.dfki.de/nifti/code/ros/stacks/nifti_drivers/trunk/nifti_robot_driver@6825 3189491a-1924-0410-a745-03ab4139b441

File: robot_model/nifti_robot.urdf (robot description, URDF)
Before this commit: robot NIFTi, 16 links, 15 joints
Links:
- link base_link: geometry visual mesh filename=package://nifti_robot_driver/robot_model/body.dae scale=0.115 0.115 0.115
- link front_left_flipper: geometry visual mesh filename=package://nifti_robot_driver/robot_model/flipper.dae scale=0.115 0.115 0.115
- link front_right_flipper: geometry visual mesh filename=package://nifti_robot_driver/robot_model/flipper.dae scale=-0.115 0.115 0.115
- link laser: geometry visual mesh filename=package://nifti_robot_driver/robot_model/laser.dae scale=0.001 0.001 0.001
- link left_track: geometry visual mesh filename=package://nifti_robot_driver/robot_model/bogie.dae scale=-0.115 0.115 0.115
- link omnicam: geometry visual mesh filename=package://nifti_robot_driver/robot_model/omnicam.stl scale=0.115 0.115 0.115
- link rear_left_flipper: geometry visual mesh filename=package://nifti_robot_driver/robot_model/flipper.dae scale=0.115 0.115 0.115
- link rear_right_flipper: geometry visual mesh filename=package://nifti_robot_driver/robot_model/flipper.dae scale=-0.115 0.115 0.115
- link right_track: geometry visual mesh filename=package://nifti_robot_driver/robot_model/bogie.dae scale=0.115 0.115 0.115
